File: Modular_Load.kicad_pcb (KiCad board)
At the start: 2 copper layers, 65 x 40 mm, 84 parts, among them J1 Conn_02x04_Odd_Even, J2 Conn_Coaxial, J3 7466203, J4 Conn_Coaxial, J5 7466203, J6 Conn_Coaxial, J7 Conn_Coaxial, Q2 IGT65R025D2, U1 ADA4807-4

Commit message: Assembly Doccumentation Updates
Parts:
- renumbered G*** to G1, G*** to G2, REF** to G3, REF** to H1, REF** to H2, REF** to H3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
Other:
- board text added: "Back Assembly Drawing"
- board text added: "Front Assembly Drawing"
